File: UART Bus Board V2.kicad_sch (KiCad schematic)
At the start: 61 parts, among them IC1 FT4232H-56Q-TRAY, J1 USB_B_Mini, J8 3.3V/5V GND TX RX TX RX TX RX, SW1 B3F-1000, U1 TC1262-33, U2 93AA46B, U3 MAX3232IPWR, U4 MAX3232IPWR, U5 M74HC595YTTR, Y1 ECS-120-8-30-JGN-TR

Commit message: Errors & warning
Fixed a couple of errors and warnings that the DRC reported.
Parts:
- added H1, H2: MountingHole, MountingHole:MountingHole_2.2mm_M2, symbol Mechanical:MountingHole
Changed lines of the file:
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@@
+    )
+  )
+  (symbol (lib_id "Mechanical:MountingHole") (at 122.428 180.848 0) (unit 1)
+    (in_bom yes) (on_board yes) (dnp no) (fields_autoplaced)
+    (property "Reference" "H1" (at 125.73 179.578 0)
+      (effects (font (size 1.27 1.27)) (justify left))
+    )
+    (property "Value" "MountingHole" (at 125.73 182.118 0)
+      (effects (font (size 1.27 1.27)) (justify left))
+    )
+    (property "Footprint" "MountingHole:MountingHole_2.2mm_M2" (at 122.428 180.848 0)
+      (effects (font (size 1.27 1.27)) hide)
+    )
+    (property "Datasheet" "~" (at 122.428 180.848 0)
+      (effects (font (size 1.27 1.27)) hide)
+    )
+    (instances
+      (project "UART Bus Board V2"
+        (path "/b854e164-eabb-4feb-95b8-76dee49c6aa9"
+          (reference "H1") (unit 1)
+        )
+      )
     )
   )
@@
         )
       )
+    )
+  )
+  (symbol (lib_id "Mechanical:MountingHole") (at 122.428 186.69 0) (unit 1)
+    (in_bom yes) (on_board yes) (dnp no) (fields_autoplaced)
+    (property "Reference" "H2" (at 125.73 185.42 0)
+      (effects (font (size 1.27 1.27)) (justify left))
+    )
+    (property "Value" "MountingHole" (at 125.73 187.96 0)
+      (effects (font (size 1.27 1.27)) (justify left))
+    )
+    (property "Footprint" "MountingHole:MountingHole_2.2mm_M2" (at 122.428 186.69 0)
+      (effects (font (size 1.27 1.27)) hide)
+    )
+    (property "Datasheet" "~" (at 122.428 186.69 0)
+      (effects (font (size 1.27 1.27)) hide)
+    )
+    (instances
+      (project "UART Bus Board V2"
+        (path "/b854e164-eabb-4feb-95b8-76dee49c6aa9"
+          (reference "H2") (unit 1)
+        )
+      )

Commit message: clearances/minimums + burried vias + PCBWay
Lowered clearances and minimums on the top fill layer
Removed three buried/hidden vias
Passing on PCBWay without issues
Parts:
- C1, C4: value 100 nF -> 1 uF
Changed lines of the file:
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@@
       (effects (font (size 1.27 1.27)) (justify left))
     )
-    (property "Value" "100 nF" (at 203.2 32.258 0)
+    (property "Value" "1 uF" (at 203.2 32.258 0)
       (effects (font (size 1.27 1.27)) (justify left))
     )
@@
   (symbol (lib_id "Device:C") (at 232.918 30.988 0) (unit 1)
     (in_bom yes) (on_board yes) (dnp no) (fields_autoplaced)
-    (property "Reference" "C1" (at 236.728 29.718 0)
-      (effects (font (size 1.27 1.27)) (justify left))
-    )
-    (property "Value" "100 nF" (at 236.728 32.258 0)
-      (effects (font (size 1.27 1.27)) (justify left))
-    )
+    (property "Reference" "C1" (at 236.22 29.718 0)
+      (effects (font (size 1.27 1.27)) (justify left))
+    )
+    (property "Value" "1 uF" (at 236.22 32.258 0)
+      (effects (font (size 1.27 1.27)) (justify left))
+    )
